File: valve_controller/valve_controller.kicad_sch (KiCad schematic)
At the start: 34 parts, among them J2 T4143512051-000, J3 M12A-04PMMP-SF8001, J4 ESP_PROG, J5 643260100604, U1 LAN8720A, U2 ADS1115IDGS, U3 MCP4728, U4 ESP32-WROOM-32, U5 LM2576S-12, U6 GP8403, U7 ADS1115IDGS, U8 LM2576S-5, U9 AP2112K-3.3, Y2 ASE-25.000MHZ-LC-T

Commit message: Fully updated DAC and regulators
Parts:
- removed C13: 10uF, Capacitor_SMD:C_0603_1608Metric, symbol SerialChiller-eagle-import:C-EUC1206
- removed C14: 0.1uF, Capacitor_SMD:C_0603_1608Metric, symbol SerialChiller-eagle-import:C-EUC1206
- removed R10, R11: 10k, Resistor_SMD:R_0603_1608Metric, symbol SerialChiller-eagle-import:R-EU_R0603
- removed R12: 100k, Resistor_SMD:R_0603_1608Metric, symbol SerialChiller-eagle-import:R-EU_R0603
- removed U3: MCP4728, Package_SO:MSOP-10_3x3mm_P0.5mm, symbol Analog_DAC:MCP4728
- removed U6: GP8403, Package_SO:MSOP-10_3x3mm_P0.5mm, symbol Analog_DAC:MCP4728
- added C10, C7, C8, C9: 100uF, Capacitor_SMD:C_0603_1608Metric, symbol SerialChiller-eagle-import:C-EUC1206
- added C12, C15, C18, C19, C21, C22, C24, C25: 0.1uF, Capacitor_SMD:C_0603_1608Metric, symbol SerialChiller-eagle-import:C-EUC1206
- added C16, C17, C20, C23: 1uF, Capacitor_SMD:C_0603_1608Metric, symbol SerialChiller-eagle-import:C-EUC1206
- added D10, D11, D2, D3, D4, D5, D6, D7, D8, D9: 1N5822, Diode_THT:D_DO-201AD_P15.24mm_Horizontal, symbol Diode:1N5822
- added J1, J10, J11, J6, J7, J8, J9: 643260100604, 643260100604:643260100604, symbol 643260100604:643260100604
- added L1, L2: MURATA_LQM21DH101M70L, symbol MURATA_LQM21DH101M70L:MURATA_LQM21DH101M70L
- added U10, U11, U12, U13: GP8403-TC50-EW, symbol GP8403-TC50-EW_C31520071_GP8403-TC50-EW_C3152007.schdoc-cache:GP8403-TC50-EW
Connections:
- net +24V: now also J3.1, U5.1 (VIN), C7.1, J1.1, J10.1, J11.1, J6.1, J7.1, J8.1, J9.1
- net +3V3: now also U8.4 (FB), C10.2, L2.2, U10.9 (A2), U11.3 (A0), U11.9 (A2), U12.4 (A1), U12.9 (A2), U13.3 (A0), U13.4 (A1), U13.9 (A2)
- net +5V: now also U5.4 (FB), C8.2, L1.2
- net AIN0_ADC1: now also J8.4
- net AIN1_ADC0: now also J1.4
- net AIN1_ADC1: now also J9.4
- net AIN2_ADC0: now also J6.4
- net AIN2_ADC1: now also J10.4
- net AIN3_ADC0: now also J7.4
- net AIN3_ADC1: now also J11.4
- net GND: now also J3.3, U5.3 (GND), U5.5 (~{ON}/OFF), U8.3 (GND), U8.5 (~{ON}/OFF), C10.1, C12.1, C15.1, C16.1, C17.1, C18.1, C19.1, C20.1, C21.1, C22.1, C23.1, C24.1, C25.1, C7.2, C8.1, C9.2, D10.2 (A), D11.2 (A), D2.2 (A), D3.2 (A), D4.2 (A), D5.2 (A), D6.2 (A), D7.2 (A), D8.2 (A), D9.2 (A), J1.3, J10.3, J11.3, J6.3, J7.3, J8.3, J9.3, U10.3 (A0), U10.4 (A1), U10.6 (GND), U11.4 (A1), U11.6 (GND), U12.3 (A0), U12.6 (GND), U13.6 (GND)
- net SCL: now also U10.1 (SCLK), U11.1 (SCLK), U12.1 (SCLK), U13.1 (SCLK)
- net SDA: now also U10.2 (SDA), U11.2 (SDA), U12.2 (SDA), U13.2 (SDA)
- net +12V: now reaches U8.1 (VIN)
- net +12V: now also C9.1, U10.5 (VCC), U11.5 (VCC), U12.5 (VCC), U13.5 (VCC)
- net at U8.2 (OUT): now also D3.1 (K), L2.1
- net at U5.2 (OUT): now also D2.1 (K), L1.1
- net ANOUT0_DAC0 renamed AOUT0_DAC0
- net AOUT0_DAC0: now also C15.2, D5.1 (K), U10.8 (VOUT0)
- new net: C23.2, U13.10 (V5V)
- new net: C20.2, U12.10 (V5V)
- new net: C17.2, U11.10 (V5V)
- new net: C16.2, U10.10 (V5V)
- new net AOUT0_DAC1: C19.2, D7.1 (K), J6.2, U11.8 (VOUT0)
- new net AOUT0_DAC2: C22.2, D9.1 (K), J8.2, U12.8 (VOUT0)
- new net AOUT0_DAC3: C25.2, D11.1 (K), J10.2, U13.8 (VOUT0)
- new net AOUT1_DAC0: C12.2, D4.1 (K), J1.2, U10.7 (VOUT1)
- new net AOUT1_DAC1: C18.2, D6.1 (K), J7.2, U11.7 (VOUT1)
- new net AOUT1_DAC2: C21.2, D8.1 (K), J9.2, U12.7 (VOUT1)
- new net AOUT1_DAC3: C24.2, D10.1 (K), J11.2, U13.7 (VOUT1)
Other:
- note added: "M12 D"
- note removed: "25MHz oscillator"
- note removed: "ADC"
- note removed: "DAC"
- note removed: "ESP32"
- note removed: "Ethernet CONNECTOR"
- note removed: "LDO 3V3"
- note removed: "Power in"
- moved on the sheet: C3, C4, C5, C6, J2, J3, J5, R1, R3, R5, R6, R7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
