File: valve_controller/valve_controller.kicad_sch (KiCad schematic)
At the start: 70 parts, among them J1 T4132512041-000, J10 M12A-05PFFP-SF8001, J12 M12A-05PFFP-SF8001, J2 20021511-00006T4LF, J3 54-00384, J4 M12A-05PFFP-SF8001, J5 M12A-05PFFP-SF8001, J6 M12A-05PFFP-SF8001, J7 M12A-05PFFP-SF8001, J8 M12A-05PFFP-SF8001, J9 M12A-05PFFP-SF8001, U1 LAN8720A, U10 ADS1115IDGS, U12 LM2576S-12, U2 ESP32-WROOM-32, U3 LM2576S-5, U4 GP8403-TC50-EW, U5 GP8403-TC50-EW, U6 AP2112K-3.3, U7 GP8403-TC50-EW, U8 ADS1115IDGS, U9 GP8403-TC50-EW, Y1 ASE-25.000MHZ-LC-T

Commit message: Routing V1
Parts:
- renumbered C27 to C10, C15 to C14, C16 to C15, C17 to C16, C18 to C17, C7 to C18, C10 to C19, C14 to C24, C24 to C25, C25 to C26, C19 to C27, C26 to C7, D9 to D10, D10 to D11, D11 to D2, D2 to D7, D7 to D8, D8 to D9, J9 to J10, J10 to J11, J12 to J4, J4 to J5, J5 to J6, J6 to J7, J7 to J8, J8 to J9, L2 to L1, L1 to L2, U9 to U10, U6 to U11, U12 to U3, U8 to U4, U4 to U5, U5 to U6, U10 to U7, U3 to U8, U7 to U9
Connections:
- net nLDAC_DAC0 is gone; now on net RXD0: U2.12 (IO27)
- net CRS_DV: now also U2.9 (IO33); no longer U2.24 (IO2)
- net MDIO: now also U2.14 (IO12); no longer U2.23 (IO15)
- net RGB_LED: now also U2.24 (IO2); no longer U2.10 (IO25)
- net RXD0: no longer U2.7 (IO35)
- net RXD1: now also U2.13 (IO14); no longer U2.6 (IO34)
- net RXER: now also U2.10 (IO25); no longer U2.26 (IO4)
- net SCL: now also U2.27 (IO16); no longer U2.36 (IO22)
- net SDA: now also U2.28 (IO17); no longer U2.37 (IO23)
- net TXD0: now also U2.16 (IO13); no longer U2.13 (IO14)
- net TXD1: now also U2.6 (IO34); no longer U2.16 (IO13)
- net TXEN: now also U2.7 (IO35); no longer U2.14 (IO12)
- net RDY_DAC0: no longer names the net of U2.11 (IO26)
- no-connect marks 22 -> 31
Other:
- moved on the sheet: R5, R6

Commit message: LED + routing V2
Parts:
- added D12, D13, D14, D15, D16, D17, D18, D19: WS2812B, LED_SMD:LED_WS2812B_PLCC4_5.0x5.0mm_P3.2mm, symbol LED:WS2812B
- added D20, D21, D22: WL-SMCW_0603, 150060VS75000:WL-SMCW_0603, symbol WL-SMCW_0603:WL-SMCW_0603
- added R8: 270, Resistor_SMD:R_0603_1608Metric, symbol SerialChiller-eagle-import:R-EU_R0603
- added R9: 10k, Resistor_SMD:R_0603_1608Metric, symbol SerialChiller-eagle-import:R-EU_R0603
- R3: value 10k -> 270
Connections:
- net +3V3: now also D12.1 (VDD), D13.1 (VDD), D14.1 (VDD), D15.1 (VDD), D16.1 (VDD), D17.1 (VDD), D18.1 (VDD), D19.1 (VDD)
- net GND: now also D12.3 (VSS), D13.3 (VSS), D14.3 (VSS), D15.3 (VSS), D16.3 (VSS), D17.3 (VSS), D18.3 (VSS), D19.3 (VSS), R8.2, R9.2
- net RGB_LED: now also U2.11 (IO26); no longer U2.24 (IO2)
- net at R3.1: now also D20.1; no longer U1.2 (LED2/~{INTSEL})
- net LED1: now reaches U1.3 (LED1/REGOFF)
- net LED1: now also D20.2
- net LED_01: now reaches D1.2 (DOUT)
- net LED_01: now also D12.4 (DIN)
- new net: D21.1, R8.1
- new net LED2: D21.2, R9.1, U1.2 (LED2/~{INTSEL})
- new net LED_12: D12.2 (DOUT), D13.4 (DIN)
- new net LED_23: D13.2 (DOUT), D14.4 (DIN)
- new net LED_34: D14.2 (DOUT), D15.4 (DIN)
- new net LED_45: D15.2 (DOUT), D16.4 (DIN)
- new net LED_56: D16.2 (DOUT), D17.4 (DIN)
- new net LED_67: D17.2 (DOUT), D18.4 (DIN)
- new net LED_78: D18.2 (DOUT), D19.4 (DIN)
- no-connect marks 31 -> 29

Commit message: tweaks for case
Parts:
- added R10: 1k, Resistor_SMD:R_0603_1608Metric, symbol SerialChiller-eagle-import:R-EU_R0603
Connections:
- net +24V: now also R10.1
- net GND: now also D22.1
- net at D22.2: now also R10.2
Changed lines of the file:
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@@
 	(symbol
 		(lib_id "power:+24V")
+		(at 280.67 222.25 0)
+		(unit 1)
+		(exclude_from_sim no)
+		(in_bom yes)
+		(on_board yes)
+		(dnp no)
+		(fields_autoplaced yes)
+		(property "Reference" "#PWR122"
+			(at 280.67 226.06 0)
+			(effects
+				(font
+					(size 1.27 1.27)
+				)
+				(hide yes)
+			)
+		)
+		(property "Value" "+24V"
+			(at 280.67 217.17 0)
+			(effects
+				(font
+					(size 1.27 1.27)
+				)
+			)
+		)
+		(property "Footprint" ""
+			(at 280.67 222.25 0)
+			(effects
+				(font
+					(size 1.27 1.27)
+				)
+				(hide yes)
+			)
+		)
+		(property "Datasheet" ""
+			(at 280.67 222.25 0)
+			(effects
+				(font
+					(size 1.27 1.27)
+				)
+				(hide yes)
+			)
+		)
+		(property "Description" "Power symbol creates a global label with name \"+24V\""
+			(at 280.67 222.25 0)
+			(effects
+				(font
+					(size 1.27 1.27)
+				)
+				(hide yes)
+			)
+		)
+		(pin "1"
+		)
+		(instances
+			(project ""
+				(path "/fabe9bf5-ed03-4936-827e-530a8ad0c6d6"
+					(reference "#PWR122")
+					(unit 1)
+				)
+			)
+		)
+	)
+	(symbol
+		(lib_id "power:+24V")
 		(at 19.05 127 0)
 		(unit 1)
@@
 	(symbol
 		(lib_id "power:GND")
+		(at 280.67 240.03 0)
+		(unit 1)
+		(exclude_from_sim no)
+		(in_bom yes)
+		(on_board yes)
+		(dnp no)
+		(fields_autoplaced yes)
+		(property "Reference" "#PWR123"
+			(at 280.67 246.38 0)
+			(effects
+				(font
+					(size 1.27 1.27)
+				)
+				(hide yes)
+			)
+		)
+		(property "Value" "GND"
+			(at 280.67 245.11 0)
+			(effects
+				(font
+					(size 1.27 1.27)
+				)
+			)
+		)
+		(property "Footprint" ""
+			(at 280.67 240.03 0)
+			(effects
+				(font
+					(size 1.27 1.27)
+				)
+				(hide yes)
+			)
+		)
+		(property "Datasheet" ""
+			(at 280.67 240.03 0)
+			(effects
+				(font
+					(size 1.27 1.27)
+				)
+				(hide yes)
+			)
+		)
+		(property "Description" "Power symbol creates a global label with name \"GND\" , ground"
+			(at 280.67 240.03 0)
+			(effects
+				(font
+					(size 1.27 1.27)
+				)
+				(hide yes)
+			)
+		)
+		(pin "1"
+		)
+		(instances
+			(project ""
+				(path "/fabe9bf5-ed03-4936-827e-530a8ad0c6d6"
+					(reference "#PWR123")
+					(unit 1)
+				)
+			)
+		)
+	)
+	(symbol
+		(lib_id "power:GND")
 		(at 205.74 48.26 0)
 		(unit 1)
@@
 					(unit 1)
 				)
+			)
+		)
+	)
+	(symbol
+		(lib_id "SerialChiller-eagle-import:R-EU_R0603")
+		(at 280.67 227.33 90)
+		(mirror x)
+		(unit 1)
+		(exclude_from_sim no)
+		(in_bom yes)
+		(on_board yes)
+		(dnp no)
+		(property "Reference" "R10"
+			(at 279.146 225.806 0)
+			(effects
+				(font
+					(size 1.4986 1.4986)
+				)
+				(justify left bottom)
+			)
+		)
+		(property "Value" "1k"
+			(at 283.718 225.044 0)
+			(effects
+				(font
+					(size 1.4986 1.4986)
+				)
+				(justify left bottom)
+			)
+		)
+		(property "Footprint" "Resistor_SMD:R_0603_1608Metric"
+			(at 280.67 227.33 0)
+			(effects
+				(font
+					(size 1.27 1.27)
+				)
+				(hide yes)
+			)
+		)
+		(property "Datasheet" ""
+			(at 280.67 227.33 0)
+			(effects
+				(font
+					(size 1.27 1.27)
+				)
+				(hide yes)
+			)
+		)
+		(property "Description" ""
+			(at 280.67 227.33 0)
+			(effects
+				(font
+					(size 1.27 1.27)
+				)
+				(hide yes)
+			)
+		)
+		(pin "1"
+		)
+		(pin "2"
+		)
+		(instances
+			(project "valve_controller"
+				(path "/fabe9bf5-ed03-4936-827e-530a8ad0c6d6"
+					(reference "R10")
+					(unit 1)
+				)

Commit message: First DRC run
Parts:
- J1: footprint CONN4_T4132512041 -> T4132512041-000:CONN4_T4132512041
- J10, J11, J4, J5, J6, J7, J8, J9: footprint CONN_SF8001_AMP -> M12A_05footprints:CONN_SF8001_AMP
- L1, L2: footprint IND_SRP6530A_BRN -> SRP6530A_100M:IND_SRP6530A_BRN
- renumbered D21 to D10, D7 to D11, D17 to D12, D22 to D14, D14 to D15, D18 to D16, D8 to D17, D9 to D18, D10 to D19, D11 to D20, D19 to D21, D15 to D22, D20 to D5, D12 to D6, D16 to D7, D5 to D8, D6 to D9, R7 to R10, R4 to R3, R5 to R4, R6 to R5, R3 to R6, R9 to R7, R10 to R9
Connections:
- no-connect marks 29 -> 30

Commit message: New ethernet and power routing
Parts:
- removed C24, C27: 22uF, Capacitor_SMD:C_0603_1608Metric, symbol SerialChiller-eagle-import:C-EUC1206
- removed D1: WS2812B, LED_SMD:LED_WS2812B_PLCC4_5.0x5.0mm_P3.2mm, symbol LED:WS2812B
- removed R10: 100k, Resistor_SMD:R_0603_1608Metric, symbol SerialChiller-eagle-import:R-EU_R0603
- removed U11: AP2112K-3.3, Package_TO_SOT_SMD:SOT-23-5, symbol Regulator_Linear:AP2112K-3.3
- added C28, C29: 1uF, Capacitor_SMD:C_0603_1608Metric, symbol SerialChiller-eagle-import:C-EUC1206
- added U12: TLV1117LV33DCYR, TLV1117LV33DCYR:VREG_TLV1117LV33DCYR, symbol TLV1117LV33DCYR:TLV1117LV33DCYR
Connections:
- net LED_01 is gone; now on net RGB_LED: D6.4 (DIN)
- net +3V3: now also C29.2, U12.2 (OUT_2), U12.4 (OUT_4)
- net +5V: now also C28.2, U12.3 (IN)
- net CRS_DV: now also U2.11 (IO26); no longer U2.9 (IO33)
- net GND: now also C28.1, C29.1, U12.1 (GND)
- net MDC: now also U2.9 (IO33); no longer U2.8 (IO32)
- net MDIO: now also U2.10 (IO25); no longer U2.14 (IO12)
- net RGB_LED: now also U2.16 (IO13); no longer U2.11 (IO26)
- net RXD0: now also U2.13 (IO14); no longer U2.12 (IO27)
- net RXD1: now also U2.14 (IO12); no longer U2.13 (IO14)
- net RXER: now also U2.12 (IO27); no longer U2.10 (IO25)
- net TXD0: now also U2.7 (IO35); no longer U2.16 (IO13)
- net TXEN: now also U2.8 (IO32); no longer U2.7 (IO35)
Other:
- note removed: "Check max freq on i2c devices"
- note removed: "LED"
- note removed: "M12 D"
- note removed: "Output connector"
- title: (none) -> Valve Controller
- moved on the sheet: C10, C12, C13, C14, C15, C16, C17, C18, C19, C20, C21, C22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
