File: valve_controller/_autosave-valve_controller.kicad_sch (KiCad schematic)
At the start: 70 parts, among them J1 T4132512041-000, J10 M12A-05PFFP-SF8001, J12 M12A-05PFFP-SF8001, J2 20021511-00006T4LF, J3 54-00384, J4 M12A-05PFFP-SF8001, J5 M12A-05PFFP-SF8001, J6 M12A-05PFFP-SF8001, J7 M12A-05PFFP-SF8001, J8 M12A-05PFFP-SF8001, J9 M12A-05PFFP-SF8001, U1 LAN8720A, U10 ADS1115IDGS, U12 LM2576S-12, U2 ESP32-WROOM-32, U3 LM2576S-5, U4 GP8403-TC50-EW, U5 GP8403-TC50-EW, U6 AP2112K-3.3, U7 GP8403-TC50-EW, U8 ADS1115IDGS, U9 GP8403-TC50-EW, Y1 ASE-25.000MHZ-LC-T

Commit message: Layout V2
Parts:
- renumbered C27 to C10, C15 to C14, C16 to C15, C17 to C16, C18 to C17, C7 to C18, C10 to C19, C14 to C24, C24 to C25, C25 to C26, C19 to C27, C26 to C7, D9 to D10, D10 to D11, D11 to D2, D2 to D7, D7 to D8, D8 to D9, J9 to J10, J10 to J11, J12 to J4, J4 to J5, J5 to J6, J6 to J7, J7 to J8, J8 to J9, L2 to L1, L1 to L2, U9 to U10, U6 to U11, U12 to U3, U8 to U4, U4 to U5, U5 to U6, U10 to U7, U3 to U8, U7 to U9
