File: valve_controller/_autosave-valve_controller.kicad_pcb (KiCad board)
At the start: 4 copper layers, 171.6 x 85 mm, 93 parts, among them J1 T4132512041-000, J10 M12A-05PFFP-SF8001, J11 M12A-05PFFP-SF8001, J2 20021511-00006T4LF, J3 54-00384, J4 M12A-05PFFP-SF8001, J5 M12A-05PFFP-SF8001, J6 M12A-05PFFP-SF8001, J7 M12A-05PFFP-SF8001, J8 M12A-05PFFP-SF8001, J9 M12A-05PFFP-SF8001, U1 LAN8720A, U10 GP8403-TC50-EW, U11 AP2112K-3.3, U2 ESP32-WROOM-32, U3 LM2576S-12, U4 ADS1115IDGS, U5 GP8403-TC50-EW, U6 GP8403-TC50-EW, U7 ADS1115IDGS, U8 LM2576S-5, U9 GP8403-TC50-EW, Y1 ASE-25.000MHZ-LC-T

Commit message: First DRC run
Parts:
- moved R6 3.46 mm to (217.1, 112.6)
- moved R8 3.46 mm to (211.6, 112.6)
- moved D10 2.50 mm to (211.6, 109.2)
- moved D14 2.50 mm to (214.4, 84.2)
- moved D5 2.50 mm to (217.2, 109.2)
- moved R7 1.35 mm to (207.5, 108.4), turned to 90 degrees
- moved ? 0.69 mm to (139.4, 101.8)
- moved REF** 0.69 mm to (139.4, 101.8)
- moved ? 0.59 mm to (139.4, 91.7)
- moved REF** 0.59 mm to (139.4, 91.7)
- renumbered D21 to D10, D7 to D11, D17 to D12, D22 to D14, D14 to D15, D18 to D16, D8 to D17, D9 to D18, D10 to D19, D11 to D20, D19 to D21, D15 to D22, D20 to D5, D12 to D6, D16 to D7, D5 to D8, D6 to D9, R7 to R10, R4 to R3, R5 to R4, R6 to R5, R3 to R6, R9 to R7, R10 to R9
Connections:
- ? pad 1: (no net) -> GND (x3)
- REF** pad 1: (no net) -> GND (x4)
Routing:
- net /ESP_IO0: track 97.7 -> 131.2 mm, vias 2 -> 3
- net GND: track 118.4 -> 125.5 mm, vias 53 -> 55
- net /SDA: track 194.3 -> 201.3 mm, vias 6 -> 7
- net /LED2: track 51.6 -> 48.2 mm
- net /LED1: track 50.9 -> 53.8 mm
- net /SCL: track 203.3 -> 205.3 mm, vias 6 -> 7
- net /RGB_LED: track 16.1 -> 17.7 mm
- net Net-(D14-Pad2): track 1.81 -> 3.23 mm
- net Net-(D5-Pad1): track 3.30 -> 4.03 mm
- net Net-(D10-Pad1): track 3.32 -> 4.00 mm
- net unconnected-(U2-IO2-Pad24): track 0.53 -> 0.00 mm
